Commit message: Config de spawn du robot effectuee

File: benrover_description/urdf/benrover.urdf (robot description, URDF)
Before this commit: robot benrover_assembly, 22 links, 21 joints
Links:
- removed link Bogie_L
- removed link Bogie_R
- removed link Cam_servo_link
- removed link Rocker_L
- removed link Rocker_R
- removed link RodEnd_L
- removed link RodEnd_R
- removed link Rod_Mid
- removed link Servo_BL
- removed link Servo_BR
- removed link Servo_FL
- removed link Servo_FR
- removed link Stepper_Link
- removed link Support_L
- removed link Support_R
- removed link Wheel_BL
- removed link Wheel_BR
- removed link Wheel_FL
- removed link Wheel_FR
- removed link Wheel_ML
- removed link Wheel_MR
- added link bogie_left, mass 0.8; collision box size=0.26 0.04 0.04; visual box size=0.26 0.04 0.04
- added link bogie_right, mass 0.8; collision box size=0.26 0.04 0.04; visual box size=0.26 0.04 0.04
- added link imu_link, mass 0.05
- added link lidar_link, mass 0.15; collision cylinder length=0.05 radius=0.04; visual cylinder length=0.05 radius=0.04
- added link rocker_left, mass 1.2; collision box size=0.40 0.04 0.04; visual box size=0.40 0.04 0.04
- added link rocker_right, mass 1.2; collision box size=0.40 0.04 0.04; visual box size=0.40 0.04 0.04
- added link steer_front_left, mass 0.1
- added link steer_front_right, mass 0.1
- added link steer_rear_left, mass 0.1
- added link steer_rear_right, mass 0.1
- added link wheel_front_left, mass 0.6; collision cylinder length=0.06 radius=0.09; visual cylinder length=0.06 radius=0.09
- added link wheel_front_right, mass 0.6; collision cylinder length=0.06 radius=0.09; visual cylinder length=0.06 radius=0.09
- added link wheel_middle_left, mass 0.6; collision cylinder length=0.06 radius=0.09; visual cylinder length=0.06 radius=0.09
- added link wheel_middle_right, mass 0.6; collision cylinder length=0.06 radius=0.09; visual cylinder length=0.06 radius=0.09
- added link wheel_rear_left, mass 0.6; collision cylinder length=0.06 radius=0.09; visual cylinder length=0.06 radius=0.09
- added link wheel_rear_right, mass 0.6; collision cylinder length=0.06 radius=0.09; visual cylinder length=0.06 radius=0.09
- link base_link: mass 7.14396598530441 -> 12.0; geometry collision box size=0.5 0.35 0.15; visual box size=0.5 0.35 0.15
Joints:
- removed joint Joint_1
- removed joint Joint_10
- removed joint Joint_12
- removed joint Joint_14
- removed joint Joint_15
- removed joint Joint_18
- removed joint Joint_19
- removed joint Joint_2
- removed joint Joint_20
- removed joint Joint_21
- removed joint Joint_22
- removed joint Joint_23
- removed joint Joint_24
- removed joint Joint_25
- removed joint Joint_26
- removed joint Joint_4
- removed joint Joint_5
- removed joint Joint_6
- removed joint Joint_7
- removed joint Joint_8
- removed joint Joint_9
- added joint bogie_left_joint: type revolute, parent rocker_left, child bogie_left, origin xyz=-0.20 0 -0.04 rpy=0 0 0, axis 0 1 0, limit lower=-0.4 upper=0.4 effort=30 velocity=1.0
- added joint bogie_right_joint: type revolute, parent rocker_right, child bogie_right, origin xyz=-0.20 0 -0.04 rpy=0 0 0, axis 0 1 0, limit lower=-0.4 upper=0.4 effort=30 velocity=1.0
- added joint imu_joint: type fixed, parent base_link, child imu_link, origin xyz=0 0 0.02 rpy=0 0 0
- added joint lidar_joint: type fixed, parent base_link, child lidar_link, origin xyz=0 0 0.15 rpy=0 0 0
- added joint rocker_left_joint: type revolute, parent base_link, child rocker_left, origin xyz=0.05 0.20 0.0 rpy=0 0 0, axis 0 1 0, limit lower=-0.6 upper=0.6 effort=50 velocity=1.0
- added joint rocker_right_joint: type revolute, parent base_link, child rocker_right, origin xyz=0.05 -0.20 0.0 rpy=0 0 0, axis 0 1 0, limit lower=-0.6 upper=0.6 effort=50 velocity=1.0
- added joint steer_front_left_joint: type revolute, parent rocker_left, child steer_front_left, origin xyz=0.20 0 -0.06 rpy=0 0 0, axis 0 0 1, limit lower=-0.6 upper=0.6 effort=10 velocity=2.0
- added joint steer_front_right_joint: type revolute, parent rocker_right, child steer_front_right, origin xyz=0.20 0 -0.06 rpy=0 0 0, axis 0 0 1, limit lower=-0.6 upper=0.6 effort=10 velocity=2.0
- added joint steer_rear_left_joint: type revolute, parent bogie_left, child steer_rear_left, origin xyz=-0.12 0 -0.08 rpy=0 0 0, axis 0 0 1, limit lower=-0.6 upper=0.6 effort=10 velocity=2.0
- added joint steer_rear_right_joint: type revolute, parent bogie_right, child steer_rear_right, origin xyz=-0.12 0 -0.08 rpy=0 0 0, axis 0 0 1, limit lower=-0.6 upper=0.6 effort=10 velocity=2.0
- added joint wheel_front_left_joint: type continuous, parent steer_front_left, child wheel_front_left, origin xyz=0 0 0 rpy=0 0 0, axis 0 1 0
- added joint wheel_front_right_joint: type continuous, parent steer_front_right, child wheel_front_right, origin xyz=0 0 0 rpy=0 0 0, axis 0 1 0
- added joint wheel_middle_left_joint: type continuous, parent bogie_left, child wheel_middle_left, origin xyz=0.12 0 -0.08 rpy=0 0 0, axis 0 1 0
- added joint wheel_middle_right_joint: type continuous, parent bogie_right, child wheel_middle_right, origin xyz=0.12 0 -0.08 rpy=0 0 0, axis 0 1 0
- added joint wheel_rear_left_joint: type continuous, parent steer_rear_left, child wheel_rear_left, origin xyz=0 0 0 rpy=0 0 0, axis 0 1 0
- added joint wheel_rear_right_joint: type continuous, parent steer_rear_right, child wheel_rear_right, origin xyz=0 0 0 rpy=0 0 0, axis 0 1 0

Commit message: Implemeentation du mapping node

File: benrover_description/urdf/benrover.urdf (robot description, URDF)
Before this commit: robot benrover_skeleton, 17 links, 16 joints
Joints:
- joint steer_front_left_joint: origin xyz=0.20 0 -0.06 rpy=0 0 0 -> xyz=0.20 0 -0.12 rpy=0 0 0
- joint steer_front_right_joint: origin xyz=0.20 0 -0.06 rpy=0 0 0 -> xyz=0.20 0 -0.12 rpy=0 0 0

Commit message: Update 1 du mapping node

File: benrover_description/urdf/benrover.urdf (robot description, URDF)
Before this commit: robot benrover_skeleton, 17 links, 16 joints
Joints:
- joint rocker_left_joint: type revolute -> fixed
- joint rocker_right_joint: type revolute -> fixed
- joint steer_front_left_joint: axis 0 0 1 -> (none); limit lower=-0.6 upper=0.6 effort=10 velocity=2.0 -> (none); type revolute -> fixed
- joint steer_front_right_joint: axis 0 0 1 -> (none); limit lower=-0.6 upper=0.6 effort=10 velocity=2.0 -> (none); type revolute -> fixed
- joint steer_rear_left_joint: axis 0 0 1 -> (none); limit lower=-0.6 upper=0.6 effort=10 velocity=2.0 -> (none); type revolute -> fixed
- joint steer_rear_right_joint: axis 0 0 1 -> (none); limit lower=-0.6 upper=0.6 effort=10 velocity=2.0 -> (none); type revolute -> fixed
